Commit message: v0 family related files

File: rma_sb_ig/resources/robots/v0variants/urdf/v0Seven.urdf (robot description, URDF)
Before this commit: robot v0, 21 links, 20 joints
Links:
- added link l2_segment_1, mass 5.12; collision box size=0.1 0.1 0.2; visual box size=0.1 0.1 0.2
- added link l2_segment_2_HIP, mass 15.36; collision box size=0.1 0.6 0.1; visual box size=0.1 0.6 0.1
- added link l2_segment_3_THIGH, mass 17.92; collision box size=0.1 0.1 0.7; visual box size=0.1 0.1 0.7
- added link l2_segment_4_FOOT, mass 10.24; collision box size=0.1 0.1 0.4; visual box size=0.1 0.1 0.4
- added link r2_segment_1, mass 5.12; collision box size=0.1 0.1 0.2; visual box size=0.1 0.1 0.2
- added link r2_segment_2_HIP, mass 15.36; collision box size=0.1 0.6 0.1; visual box size=0.1 0.6 0.1
- added link r2_segment_3_THIGH, mass 17.92; collision box size=0.1 0.1 0.7; visual box size=0.1 0.1 0.7
- added link r2_segment_4_FOOT, mass 10.24; collision box size=0.1 0.1 0.4; visual box size=0.1 0.1 0.4
Joints:
- added joint l2_base_to_joint_1: type fixed, parent body, child l2_segment_1, origin xyz=0 0.1 0.75 rpy=0 0 0
- added joint l2_joint_1_to_2: type revolute, parent l2_segment_1, child l2_segment_2_HIP, origin xyz=0 0 0.25 rpy=0 0 0, axis 0.0 0.0 1.0, limit lower=-1.2 upper=1.2 effort=2048 velocity=20
- added joint l2_joint_2_to_3: type revolute, parent l2_segment_2_HIP, child l2_segment_3_THIGH, origin xyz=-0.1 0.5 0 rpy=0 0 0, axis 1.0 0.0 0.0, limit lower=-0.2 upper=0.75 effort=2048 velocity=20
- added joint l2_joint_3_to_4_FOOT: type revolute, parent l2_segment_3_THIGH, child l2_segment_4_FOOT, origin xyz=0.1 0 -0.55 rpy=0 0 0, axis 1.0 0.0 0.0, limit lower=-0.2 upper=0.5 effort=2048 velocity=20
- added joint r2_base_to_joint_1: type fixed, parent body, child r2_segment_1, origin xyz=0 -0.1 0.75 rpy=0 0 0
- added joint r2_joint_1_to_2: type revolute, parent r2_segment_1, child r2_segment_2_HIP, origin xyz=0 0 0.25 rpy=0 0 0, axis 0.0 0.0 1.0, limit lower=-1.2 upper=1.2 effort=2048 velocity=20
- added joint r2_joint_2_to_3: type revolute, parent r2_segment_2_HIP, child r2_segment_3_THIGH, origin xyz=-0.1 -0.5 0 rpy=0 0 0, axis 1.0 0.0 0.0, limit lower=-0.75 upper=0.2 effort=2048 velocity=20
- added joint r2_joint_3_to_4_FOOT: type revolute, parent r2_segment_3_THIGH, child r2_segment_4_FOOT, origin xyz=0.1 0 -0.55 rpy=0 0 0, axis 1.0 0.0 0.0, limit lower=-0.5 upper=0.2 effort=2048 velocity=20

File: rma_sb_ig/resources/robots/v0variants/urdf/v0Seven.urdf.xacro (robot description, xacro)
@@ -103,7 +103,7 @@
 		<origin xyz="0.35 0.1 .75" rpy="0 0 0" />
 	</xacro:leg>
-<!--	<xacro:leg name="l2" reflect="1">-->
-<!--		<origin xyz="0 0.1 1.05" rpy="0 0 0" />-->
-<!--	</xacro:leg>-->
+	<xacro:leg name="l2" reflect="1">
+		<origin xyz="0 0.1 0.75" rpy="0 0 0" />
+	</xacro:leg>
 	<xacro:leg name="l3" reflect="1">
 		<origin xyz="-0.5 0.1 .75" rpy="0 0 0" />
@@ -112,7 +112,7 @@
 		<origin xyz="0.35 -0.1 .75" rpy="0 0 0" />
 	</xacro:leg>
-<!--	<xacro:leg name="r2" reflect="-1">-->
-<!--		<origin xyz="0 -0.1 1.05" rpy="0 0 0" />-->
-<!--	</xacro:leg>-->
+	<xacro:leg name="r2" reflect="-1">
+		<origin xyz="0 -0.1 0.75" rpy="0 0 0" />
+	</xacro:leg>
 	<xacro:leg name="r3" reflect="-1">
 		<origin xyz="-0.5 -0.1 .75" rpy="0 0 0" />

File: rma_sb_ig/resources/robots/v0variants/urdf/v0Three.urdf (robot description, URDF)
Before this commit: robot v0, 21 links, 20 joints
Links:
- removed link l1_segment_1
- removed link l1_segment_2_HIP
- removed link l1_segment_3_THIGH
- removed link l1_segment_4_FOOT
- removed link l3_segment_1
- removed link l3_segment_2_HIP
- removed link l3_segment_3_THIGH
- removed link l3_segment_4_FOOT
- removed link r1_segment_1
- removed link r1_segment_2_HIP
- removed link r1_segment_3_THIGH
- removed link r1_segment_4_FOOT
- removed link r3_segment_1
- removed link r3_segment_2_HIP
- removed link r3_segment_3_THIGH
- removed link r3_segment_4_FOOT
- added link l2_segment_1, mass 5.12; collision box size=0.1 0.1 0.2; visual box size=0.1 0.1 0.2
- added link l2_segment_2_HIP, mass 15.36; collision box size=0.1 0.6 0.1; visual box size=0.1 0.6 0.1
- added link l2_segment_3_THIGH, mass 17.92; collision box size=0.1 0.1 0.7; visual box size=0.1 0.1 0.7
- added link l2_segment_4_FOOT, mass 10.24; collision box size=0.1 0.1 0.4; visual box size=0.1 0.1 0.4
- added link r2_segment_1, mass 5.12; collision box size=0.1 0.1 0.2; visual box size=0.1 0.1 0.2
- added link r2_segment_2_HIP, mass 15.36; collision box size=0.1 0.6 0.1; visual box size=0.1 0.6 0.1
- added link r2_segment_3_THIGH, mass 17.92; collision box size=0.1 0.1 0.7; visual box size=0.1 0.1 0.7
- added link r2_segment_4_FOOT, mass 10.24; collision box size=0.1 0.1 0.4; visual box size=0.1 0.1 0.4
Joints:
- removed joint l1_base_to_joint_1
- removed joint l1_joint_1_to_2
- removed joint l1_joint_2_to_3
- removed joint l1_joint_3_to_4_FOOT
- removed joint l3_base_to_joint_1
- removed joint l3_joint_1_to_2
- removed joint l3_joint_2_to_3
- removed joint l3_joint_3_to_4_FOOT
- removed joint r1_base_to_joint_1
- removed joint r1_joint_1_to_2
- removed joint r1_joint_2_to_3
- removed joint r1_joint_3_to_4_FOOT
- removed joint r3_base_to_joint_1
- removed joint r3_joint_1_to_2
- removed joint r3_joint_2_to_3
- removed joint r3_joint_3_to_4_FOOT
- added joint l2_base_to_joint_1: type fixed, parent body, child l2_segment_1, origin xyz=0 0.1 0.75 rpy=0 0 0
- added joint l2_joint_1_to_2: type revolute, parent l2_segment_1, child l2_segment_2_HIP, origin xyz=0 0 0.25 rpy=0 0 0, axis 0.0 0.0 1.0, limit lower=-1.2 upper=1.2 effort=2048 velocity=20
- added joint l2_joint_2_to_3: type revolute, parent l2_segment_2_HIP, child l2_segment_3_THIGH, origin xyz=-0.1 0.5 0 rpy=0 0 0, axis 1.0 0.0 0.0, limit lower=-0.2 upper=0.75 effort=2048 velocity=20
- added joint l2_joint_3_to_4_FOOT: type revolute, parent l2_segment_3_THIGH, child l2_segment_4_FOOT, origin xyz=0.1 0 -0.55 rpy=0 0 0, axis 1.0 0.0 0.0, limit lower=-0.2 upper=0.5 effort=2048 velocity=20
- added joint r2_base_to_joint_1: type fixed, parent body, child r2_segment_1, origin xyz=0 -0.1 0.75 rpy=0 0 0
- added joint r2_joint_1_to_2: type revolute, parent r2_segment_1, child r2_segment_2_HIP, origin xyz=0 0 0.25 rpy=0 0 0, axis 0.0 0.0 1.0, limit lower=-1.2 upper=1.2 effort=2048 velocity=20
- added joint r2_joint_2_to_3: type revolute, parent r2_segment_2_HIP, child r2_segment_3_THIGH, origin xyz=-0.1 -0.5 0 rpy=0 0 0, axis 1.0 0.0 0.0, limit lower=-0.75 upper=0.2 effort=2048 velocity=20
- added joint r2_joint_3_to_4_FOOT: type revolute, parent r2_segment_3_THIGH, child r2_segment_4_FOOT, origin xyz=0.1 0 -0.55 rpy=0 0 0, axis 1.0 0.0 0.0, limit lower=-0.5 upper=0.2 effort=2048 velocity=20

File: rma_sb_ig/resources/robots/v0variants/urdf/v0Three.urdf.xacro (robot description, xacro)
@@ -100,22 +100,22 @@
 		</xacro:mybox>
 	</link>
-	<xacro:leg name="l1" reflect="1">
-		<origin xyz="0.35 0.1 .75" rpy="0 0 0" />
+<!--	<xacro:leg name="l1" reflect="1">-->
+<!--		<origin xyz="0.35 0.1 .75" rpy="0 0 0" />-->
+<!--	</xacro:leg>-->
+	<xacro:leg name="l2" reflect="1">
+		<origin xyz="0 0.1 0.75" rpy="0 0 0" />
 	</xacro:leg>
-<!--	<xacro:leg name="l2" reflect="1">-->
-<!--		<origin xyz="0 0.1 1.05" rpy="0 0 0" />-->
+<!--	<xacro:leg name="l3" reflect="1">-->
+<!--		<origin xyz="-0.5 0.1 .75" rpy="0 0 0" />-->
 <!--	</xacro:leg>-->
-	<xacro:leg name="l3" reflect="1">
-		<origin xyz="-0.5 0.1 .75" rpy="0 0 0" />
+<!--	<xacro:leg name="r1" reflect="-1">-->
+<!--		<origin xyz="0.35 -0.1 .75" rpy="0 0 0" />-->
+<!--	</xacro:leg>-->
+	<xacro:leg name="r2" reflect="-1">
+		<origin xyz="0 -0.1 0.75" rpy="0 0 0" />
 	</xacro:leg>
-	<xacro:leg name="r1" reflect="-1">
-		<origin xyz="0.35 -0.1 .75" rpy="0 0 0" />
-	</xacro:leg>
-<!--	<xacro:leg name="r2" reflect="-1">-->
-<!--		<origin xyz="0 -0.1 1.05" rpy="0 0 0" />-->
+<!--	<xacro:leg name="r3" reflect="-1">-->
+<!--		<origin xyz="-0.5 -0.1 .75" rpy="0 0 0" />-->
 <!--	</xacro:leg>-->
-	<xacro:leg name="r3" reflect="-1">
-		<origin xyz="-0.5 -0.1 .75" rpy="0 0 0" />
-	</xacro:leg>
 	<xacro:leg name="r4" reflect="-1">
 		<origin xyz="0.5 -0. .75" rpy="0 0 1.57" />
