Commit message: Variable robots

File: rma_sb_ig/resources/robots/v0variants/urdf/v0_template.urdf.xacro (robot description, xacro)
@@ -1,5 +1,5 @@
 <?xml version="1.0"?>
 <robot xmlns:xacro="http://www.ros.org/wiki/xacro" name="v0">
-	<xacro:macro name="box" params="sizeX sizeY sizeZ color *origin">
+	<xacro:macro name="mybox" params="sizeX sizeY sizeZ color *origin">
 		<visual>
 			<geometry>
@@ -27,7 +27,7 @@
 	<xacro:macro name="leg" params="name reflect *origin">
 		<link name="${name}_segment_1">
-			<xacro:box sizeX="0.1" sizeY="0.1" sizeZ="0.2" color="white">
+			<xacro:mybox sizeX="0.1" sizeY="0.1" sizeZ="0.2" color="white">
 				<origin xyz="0 0 0.1" rpy="0 0 0" />
-			</xacro:box>
+			</xacro:mybox>
 		</link>
 		<joint name="${name}_base_to_joint_1" type="fixed">
@@ -37,7 +37,7 @@
 		</joint>
 		<link name="${name}_segment_2_HIP">
-			<xacro:box sizeX="0.1" sizeY="0.6" sizeZ="0.1" color="yellow">
+			<xacro:mybox sizeX="0.1" sizeY="0.6" sizeZ="0.1" color="yellow">
 				<origin xyz="0 ${reflect*0.25} 0" rpy="0 0 0" />
-			</xacro:box>
+			</xacro:mybox>
 		</link>
 		<joint name="${name}_joint_1_to_2" type="revolute">
@@ -49,7 +49,7 @@
 		</joint>
 		<link name="${name}_segment_3_THIGH">
-			<xacro:box sizeX="0.1" sizeY="0.1" sizeZ="0.7" color="red">
+			<xacro:mybox sizeX="0.1" sizeY="0.1" sizeZ="0.7" color="red">
 				<origin xyz="0 0 -0.3" rpy="0 0 0" />
-			</xacro:box>
+			</xacro:mybox>
 		</link>
 		<joint name="${name}_joint_2_to_3" type="revolute">
@@ -66,7 +66,7 @@
 		</joint>
 		<link name="${name}_segment_4_FOOT">
-			<xacro:box sizeX="0.1" sizeY="0.1" sizeZ="0.4" color="yellow">
+			<xacro:mybox sizeX="0.1" sizeY="0.1" sizeZ="0.4" color="yellow">
 				<origin xyz="0 0 -0.2" rpy="0 0 0" />
-			</xacro:box>
+			</xacro:mybox>
 		</link>
 		<joint name="${name}_joint_3_to_4_FOOT" type="revolute">
@@ -96,7 +96,7 @@
 	</material>
 	<link name="body">
-		<xacro:box sizeX="1.3" sizeY="0.3" sizeZ="0.1" color="grey">
+		<xacro:mybox sizeX="1.3" sizeY="0.3" sizeZ="0.1" color="grey">
 			<origin xyz="0 0 0.7" rpy="0 0 0" />
-		</xacro:box>
+		</xacro:mybox>
 	</link>
 <!--	<xacro:leg name="l1" reflect="1">-->
