Commit message: last changes

File: rma_sb_ig/resources/robots/soto_2/soto_gripper.urdf (robot description, URDF)
Before this commit: robot soto_2_1, 79 links, 78 joints
Links:
- link cylinder_left_10: mass 0.3 -> 0.15
- link cylinder_left_11: mass 0.3 -> 0.15
- link cylinder_left_12: mass 0.3 -> 0.15
- link cylinder_left_13: mass 0.3 -> 0.15
- link cylinder_left_14: mass 0.3 -> 0.15
- link cylinder_left_15: mass 0.3 -> 0.15
- link cylinder_left_16: mass 0.3 -> 0.15
- link cylinder_left_17: mass 0.3 -> 0.15
- link cylinder_left_18: mass 0.3 -> 0.15
- link cylinder_left_19: mass 0.3 -> 0.15
- link cylinder_left_20: mass 0.3 -> 0.15
- link cylinder_left_21: mass 0.3 -> 0.15
- link cylinder_left_22: mass 0.3 -> 0.15
- link cylinder_left_23: mass 0.3 -> 0.15
- link cylinder_left_24: mass 0.3 -> 0.15
- link cylinder_left_25: mass 0.3 -> 0.15
- link cylinder_left_26: mass 0.3 -> 0.15
- link cylinder_left_27: mass 0.3 -> 0.15
- link cylinder_left_28: mass 0.3 -> 0.15
- link cylinder_left_29: mass 0.3 -> 0.15
- link cylinder_left_30: mass 0.3 -> 0.15
- link cylinder_left_31: mass 0.3 -> 0.15
- link cylinder_left_4: mass 0.3 -> 0.15
- link cylinder_left_5: mass 0.3 -> 0.15
- link cylinder_left_6: mass 0.3 -> 0.15
- link cylinder_left_7: mass 0.3 -> 0.15
- link cylinder_left_8: mass 0.3 -> 0.15
- link cylinder_left_9: mass 0.3 -> 0.15
- link cylinder_right_10: mass 0.3 -> 0.15
- link cylinder_right_11: mass 0.3 -> 0.15
- link cylinder_right_12: mass 0.3 -> 0.15
- link cylinder_right_13: mass 0.3 -> 0.15
- link cylinder_right_14: mass 0.3 -> 0.15
- link cylinder_right_15: mass 0.3 -> 0.15
- link cylinder_right_16: mass 0.3 -> 0.15
- link cylinder_right_17: mass 0.3 -> 0.15
- link cylinder_right_18: mass 0.3 -> 0.15
- link cylinder_right_19: mass 0.3 -> 0.15
- link cylinder_right_20: mass 0.3 -> 0.15
- link cylinder_right_21: mass 0.3 -> 0.15
- link cylinder_right_22: mass 0.3 -> 0.15
- link cylinder_right_23: mass 0.3 -> 0.15
- link cylinder_right_24: mass 0.3 -> 0.15
- link cylinder_right_25: mass 0.3 -> 0.15
- link cylinder_right_26: mass 0.3 -> 0.15
- link cylinder_right_27: mass 0.3 -> 0.15
- link cylinder_right_28: mass 0.3 -> 0.15
- link cylinder_right_29: mass 0.3 -> 0.15
- link cylinder_right_30: mass 0.3 -> 0.15
- link cylinder_right_31: mass 0.3 -> 0.15
- link cylinder_right_4: mass 0.3 -> 0.15
- link cylinder_right_5: mass 0.3 -> 0.15
- link cylinder_right_6: mass 0.3 -> 0.15
- link cylinder_right_7: mass 0.3 -> 0.15
- link cylinder_right_8: mass 0.3 -> 0.15
- link cylinder_right_9: mass 0.3 -> 0.15
Joints:
- joint cylinder_left_10_to_belt: limit lower=-100 upper=100 effort=100 velocity=100 -> lower=-10 upper=10 effort=10 velocity=10
- joint cylinder_left_11_to_belt: limit lower=-100 upper=100 effort=100 velocity=100 -> lower=-10 upper=10 effort=10 velocity=10
- joint cylinder_left_12_to_belt: limit lower=-100 upper=100 effort=100 velocity=100 -> lower=-10 upper=10 effort=10 velocity=10
- joint cylinder_left_13_to_belt: limit lower=-100 upper=100 effort=100 velocity=100 -> lower=-10 upper=10 effort=10 velocity=10
- joint cylinder_left_14_to_belt: limit lower=-100 upper=100 effort=100 velocity=100 -> lower=-10 upper=10 effort=10 velocity=10
- joint cylinder_left_15_to_belt: limit lower=-100 upper=100 effort=100 velocity=100 -> lower=-10 upper=10 effort=10 velocity=10
- joint cylinder_left_16_to_belt: limit lower=-100 upper=100 effort=100 velocity=100 -> lower=-10 upper=10 effort=10 velocity=10
- joint cylinder_left_17_to_belt: limit lower=-100 upper=100 effort=100 velocity=100 -> lower=-10 upper=10 effort=10 velocity=10
- joint cylinder_left_18_to_belt: limit lower=-100 upper=100 effort=100 velocity=100 -> lower=-10 upper=10 effort=10 velocity=10
- joint cylinder_left_19_to_belt: limit lower=-100 upper=100 effort=100 velocity=100 -> lower=-10 upper=10 effort=10 velocity=10
- joint cylinder_left_20_to_belt: limit lower=-100 upper=100 effort=100 velocity=100 -> lower=-10 upper=10 effort=10 velocity=10
- joint cylinder_left_21_to_belt: limit lower=-100 upper=100 effort=100 velocity=100 -> lower=-10 upper=10 effort=10 velocity=10
- joint cylinder_left_22_to_belt: limit lower=-100 upper=100 effort=100 velocity=100 -> lower=-10 upper=10 effort=10 velocity=10
- joint cylinder_left_23_to_belt: limit lower=-100 upper=100 effort=100 velocity=100 -> lower=-10 upper=10 effort=10 velocity=10
- joint cylinder_left_24_to_belt: limit lower=-100 upper=100 effort=100 velocity=100 -> lower=-10 upper=10 effort=10 velocity=10
- joint cylinder_left_25_to_belt: limit lower=-100 upper=100 effort=100 velocity=100 -> lower=-10 upper=10 effort=10 velocity=10
- joint cylinder_left_26_to_belt: limit lower=-100 upper=100 effort=100 velocity=100 -> lower=-10 upper=10 effort=10 velocity=10
- joint cylinder_left_27_to_belt: limit lower=-100 upper=100 effort=100 velocity=100 -> lower=-10 upper=10 effort=10 velocity=10
- joint cylinder_left_28_to_belt: limit lower=-100 upper=100 effort=100 velocity=100 -> lower=-10 upper=10 effort=10 velocity=10
- joint cylinder_left_29_to_belt: limit lower=-100 upper=100 effort=100 velocity=100 -> lower=-10 upper=10 effort=10 velocity=10
- joint cylinder_left_30_to_belt: limit lower=-100 upper=100 effort=100 velocity=100 -> lower=-10 upper=10 effort=10 velocity=10
- joint cylinder_left_31_to_belt: limit lower=-100 upper=100 effort=100 velocity=100 -> lower=-10 upper=10 effort=10 velocity=10
- joint cylinder_left_4_to_belt: limit lower=-100 upper=100 effort=100 velocity=100 -> lower=-10 upper=10 effort=10 velocity=10
- joint cylinder_left_5_to_belt: limit lower=-100 upper=100 effort=100 velocity=100 -> lower=-10 upper=10 effort=10 velocity=10
- joint cylinder_left_6_to_belt: limit lower=-100 upper=100 effort=100 velocity=100 -> lower=-10 upper=10 effort=10 velocity=10
- joint cylinder_left_7_to_belt: limit lower=-100 upper=100 effort=100 velocity=100 -> lower=-10 upper=10 effort=10 velocity=10
- joint cylinder_left_8_to_belt: limit lower=-100 upper=100 effort=100 velocity=100 -> lower=-10 upper=10 effort=10 velocity=10
- joint cylinder_left_9_to_belt: limit lower=-100 upper=100 effort=100 velocity=100 -> lower=-10 upper=10 effort=10 velocity=10
- joint cylinder_right_10_to_belt: limit lower=-100 upper=100 effort=100 velocity=100 -> lower=-10 upper=10 effort=10 velocity=10
- joint cylinder_right_11_to_belt: limit lower=-100 upper=100 effort=100 velocity=100 -> lower=-10 upper=10 effort=10 velocity=10
- joint cylinder_right_12_to_belt: limit lower=-100 upper=100 effort=100 velocity=100 -> lower=-10 upper=10 effort=10 velocity=10
- joint cylinder_right_13_to_belt: limit lower=-100 upper=100 effort=100 velocity=100 -> lower=-10 upper=10 effort=10 velocity=10
- joint cylinder_right_14_to_belt: limit lower=-100 upper=100 effort=100 velocity=100 -> lower=-10 upper=10 effort=10 velocity=10
- joint cylinder_right_15_to_belt: limit lower=-100 upper=100 effort=100 velocity=100 -> lower=-10 upper=10 effort=10 velocity=10
- joint cylinder_right_16_to_belt: limit lower=-100 upper=100 effort=100 velocity=100 -> lower=-10 upper=10 effort=10 velocity=10
- joint cylinder_right_17_to_belt: limit lower=-100 upper=100 effort=100 velocity=100 -> lower=-10 upper=10 effort=10 velocity=10
- joint cylinder_right_18_to_belt: limit lower=-100 upper=100 effort=100 velocity=100 -> lower=-10 upper=10 effort=10 velocity=10
- joint cylinder_right_19_to_belt: limit lower=-100 upper=100 effort=100 velocity=100 -> lower=-10 upper=10 effort=10 velocity=10
- joint cylinder_right_20_to_belt: limit lower=-100 upper=100 effort=100 velocity=100 -> lower=-10 upper=10 effort=10 velocity=10
- joint cylinder_right_21_to_belt: limit lower=-100 upper=100 effort=100 velocity=100 -> lower=-10 upper=10 effort=10 velocity=10
- joint cylinder_right_22_to_belt: limit lower=-100 upper=100 effort=100 velocity=100 -> lower=-10 upper=10 effort=10 velocity=10
- joint cylinder_right_23_to_belt: limit lower=-100 upper=100 effort=100 velocity=100 -> lower=-10 upper=10 effort=10 velocity=10
- joint cylinder_right_24_to_belt: limit lower=-100 upper=100 effort=100 velocity=100 -> lower=-10 upper=10 effort=10 velocity=10
- joint cylinder_right_25_to_belt: limit lower=-100 upper=100 effort=100 velocity=100 -> lower=-10 upper=10 effort=10 velocity=10
- joint cylinder_right_26_to_belt: limit lower=-100 upper=100 effort=100 velocity=100 -> lower=-10 upper=10 effort=10 velocity=10
- joint cylinder_right_27_to_belt: limit lower=-100 upper=100 effort=100 velocity=100 -> lower=-10 upper=10 effort=10 velocity=10
- joint cylinder_right_28_to_belt: limit lower=-100 upper=100 effort=100 velocity=100 -> lower=-10 upper=10 effort=10 velocity=10
- joint cylinder_right_29_to_belt: limit lower=-100 upper=100 effort=100 velocity=100 -> lower=-10 upper=10 effort=10 velocity=10
- joint cylinder_right_30_to_belt: limit lower=-100 upper=100 effort=100 velocity=100 -> lower=-10 upper=10 effort=10 velocity=10
- joint cylinder_right_31_to_belt: limit lower=-100 upper=100 effort=100 velocity=100 -> lower=-10 upper=10 effort=10 velocity=10
- joint cylinder_right_4_to_belt: limit lower=-100 upper=100 effort=100 velocity=100 -> lower=-10 upper=10 effort=10 velocity=10
- joint cylinder_right_5_to_belt: limit lower=-100 upper=100 effort=100 velocity=100 -> lower=-10 upper=10 effort=10 velocity=10
- joint cylinder_right_6_to_belt: limit lower=-100 upper=100 effort=100 velocity=100 -> lower=-10 upper=10 effort=10 velocity=10
- joint cylinder_right_7_to_belt: limit lower=-100 upper=100 effort=100 velocity=100 -> lower=-10 upper=10 effort=10 velocity=10
- joint cylinder_right_8_to_belt: limit lower=-100 upper=100 effort=100 velocity=100 -> lower=-10 upper=10 effort=10 velocity=10
- joint cylinder_right_9_to_belt: limit lower=-100 upper=100 effort=100 velocity=100 -> lower=-10 upper=10 effort=10 velocity=10

Commit message: major add : conveyor_belt

File: rma_sb_ig/resources/robots/soto_2/soto_gripper.urdf (robot description, URDF)
Before this commit: robot soto_2_1, 79 links, 78 joints
Links:
- removed link cylinder_left_10
- removed link cylinder_left_11
- removed link cylinder_left_12
- removed link cylinder_left_13
- removed link cylinder_left_14
- removed link cylinder_left_15
- removed link cylinder_left_16
- removed link cylinder_left_17
- removed link cylinder_left_18
- removed link cylinder_left_19
- removed link cylinder_left_20
- removed link cylinder_left_21
- removed link cylinder_left_22
- removed link cylinder_left_23
- removed link cylinder_left_24
- removed link cylinder_left_25
- removed link cylinder_left_26
- removed link cylinder_left_27
- removed link cylinder_left_28
- removed link cylinder_left_29
- removed link cylinder_left_30
- removed link cylinder_left_31
- removed link cylinder_left_4
- removed link cylinder_left_5
- removed link cylinder_left_6
- removed link cylinder_left_7
- removed link cylinder_left_8
- removed link cylinder_left_9
- removed link cylinder_right_10
- removed link cylinder_right_11
- removed link cylinder_right_12
- removed link cylinder_right_13
- removed link cylinder_right_14
- removed link cylinder_right_15
- removed link cylinder_right_16
- removed link cylinder_right_17
- removed link cylinder_right_18
- removed link cylinder_right_19
- removed link cylinder_right_20
- removed link cylinder_right_21
- removed link cylinder_right_22
- removed link cylinder_right_23
- removed link cylinder_right_24
- removed link cylinder_right_25
- removed link cylinder_right_26
- removed link cylinder_right_27
- removed link cylinder_right_28
- removed link cylinder_right_29
- removed link cylinder_right_30
- removed link cylinder_right_31
- removed link cylinder_right_4
- removed link cylinder_right_5
- removed link cylinder_right_6
- removed link cylinder_right_7
- removed link cylinder_right_8
- removed link cylinder_right_9
- added link left_conveyor_belt, mass 2.0; collision box size=2 0.05 0.005; visual box size=2 0.05 0.005
- added link right_conveyor_belt, mass 2.0; collision box size=2 0.05 0.005; visual box size=2.0 0.05 0.005
Joints:
- removed joint cylinder_left_10_to_belt
- removed joint cylinder_left_11_to_belt
- removed joint cylinder_left_12_to_belt
- removed joint cylinder_left_13_to_belt
- removed joint cylinder_left_14_to_belt
- removed joint cylinder_left_15_to_belt
- removed joint cylinder_left_16_to_belt
- removed joint cylinder_left_17_to_belt
- removed joint cylinder_left_18_to_belt
- removed joint cylinder_left_19_to_belt
- removed joint cylinder_left_20_to_belt
- removed joint cylinder_left_21_to_belt
- removed joint cylinder_left_22_to_belt
- removed joint cylinder_left_23_to_belt
- removed joint cylinder_left_24_to_belt
- removed joint cylinder_left_25_to_belt
- removed joint cylinder_left_26_to_belt
- removed joint cylinder_left_27_to_belt
- removed joint cylinder_left_28_to_belt
- removed joint cylinder_left_29_to_belt
- removed joint cylinder_left_30_to_belt
- removed joint cylinder_left_31_to_belt
- removed joint cylinder_left_4_to_belt
- removed joint cylinder_left_5_to_belt
- removed joint cylinder_left_6_to_belt
- removed joint cylinder_left_7_to_belt
- removed joint cylinder_left_8_to_belt
- removed joint cylinder_left_9_to_belt
- removed joint cylinder_right_10_to_belt
- removed joint cylinder_right_11_to_belt
- removed joint cylinder_right_12_to_belt
- removed joint cylinder_right_13_to_belt
- removed joint cylinder_right_14_to_belt
- removed joint cylinder_right_15_to_belt
- removed joint cylinder_right_16_to_belt
- removed joint cylinder_right_17_to_belt
- removed joint cylinder_right_18_to_belt
- removed joint cylinder_right_19_to_belt
- removed joint cylinder_right_20_to_belt
- removed joint cylinder_right_21_to_belt
- removed joint cylinder_right_22_to_belt
- removed joint cylinder_right_23_to_belt
- removed joint cylinder_right_24_to_belt
- removed joint cylinder_right_25_to_belt
- removed joint cylinder_right_26_to_belt
- removed joint cylinder_right_27_to_belt
- removed joint cylinder_right_28_to_belt
- removed joint cylinder_right_29_to_belt
- removed joint cylinder_right_30_to_belt
- removed joint cylinder_right_31_to_belt
- removed joint cylinder_right_4_to_belt
- removed joint cylinder_right_5_to_belt
- removed joint cylinder_right_6_to_belt
- removed joint cylinder_right_7_to_belt
- removed joint cylinder_right_8_to_belt
- removed joint cylinder_right_9_to_belt
- added joint conveyor_left_to_belt: type prismatic, parent conveyor_belt_left_foremost_link, child left_conveyor_belt, origin xyz=0.0 0.0 0.005, axis 1 0 0, limit lower=-5 upper=+5 effort=1500 velocity=0.50
- added joint conveyor_right_to_belt: type prismatic, parent conveyor_belt_right_foremost_link, child right_conveyor_belt, origin xyz=0.0 0.0 0.005, axis 1 0 0, limit lower=-5 upper=5 effort=1500 velocity=0.50

Commit message: working headless version

File: rma_sb_ig/resources/robots/soto_2/soto_gripper.urdf (robot description, URDF)
Before this commit: robot soto_2_1, 25 links, 24 joints
Links:
- link left_conveyor_belt: mass 2.0 -> 5.0
- link right_conveyor_belt: mass 2.0 -> 5.0
Joints:
- joint conveyor_left_to_belt: limit lower=-5 upper=+5 effort=1500 velocity=0.50 -> lower=-5 upper=+5 effort=150000 velocity=1
- joint conveyor_right_to_belt: limit lower=-5 upper=5 effort=1500 velocity=0.50 -> lower=-5 upper=5 effort=150000 velocity=1

Commit message: huge progess

File: rma_sb_ig/resources/robots/soto_2/soto_gripper.urdf (robot description, URDF)
Before this commit: robot soto_2_1, 25 links, 24 joints
Links:
- link left_conveyor_belt: geometry collision box size=5.0 0.05 0.005; visual box size=5.0 0.05 0.005
- link right_conveyor_belt: geometry collision box size=5.0 0.05 0.005; visual box size=5.0 0.05 0.005
Joints:
- joint conveyor_left_to_belt: limit lower=-5 upper=+5 effort=150000 velocity=1 -> lower=-10.0 upper=10.0 effort=15000.0 velocity=1
- joint conveyor_right_to_belt: limit lower=-5 upper=5 effort=150000 velocity=1 -> lower=-10.0 upper=10.0 effort=15000.0 velocity=1

Commit message: try

File: rma_sb_ig/resources/robots/soto_2/soto_gripper.urdf (robot description, URDF)
Before this commit: robot soto_2_1, 25 links, 24 joints
Links:
- link left_conveyor_belt: mass 5.0 -> 0.3; geometry collision box size=5.0 0.05 0.01; visual box size=5.0 0.05 0.01
- link right_conveyor_belt: mass 5.0 -> 0.3; geometry collision box size=5.0 0.05 0.01; visual box size=5.0 0.05 0.01
Joints:
- joint conveyor_left_to_belt: limit lower=-10.0 upper=10.0 effort=15000.0 velocity=1 -> lower=-2.5 upper=2.5 effort=10000 velocity=0.3; origin xyz=0.0 0.0 0.005 -> xyz=0.0 0.0 0.01
- joint conveyor_right_to_belt: limit lower=-10.0 upper=10.0 effort=15000.0 velocity=1 -> lower=-2.5 upper=2.5 effort=10000 velocity=0.3; origin xyz=0.0 0.0 0.005 -> xyz=0.0 0.0 0.01

Commit message: turning works

File: rma_sb_ig/resources/robots/soto_2/soto_gripper.urdf (robot description, URDF)
Before this commit: robot soto_2_1, 25 links, 24 joints
Joints:
- joint conveyor_left_to_belt: limit lower=-2.5 upper=2.5 effort=10000 velocity=0.3 -> lower=-2.5 upper=2.5 effort=1000 velocity=0.3
- joint conveyor_right_to_belt: limit lower=-2.5 upper=2.5 effort=10000 velocity=0.3 -> lower=-2.5 upper=2.5 effort=1000 velocity=0.3
- joint gripper_rotate: axis 0 0 1 -> (none); limit lower=-3.22886 upper=1.65806 effort=32.11 velocity=3.72802 -> (none); type revolute -> fixed
- joint gripper_y_left: limit lower=0.002 upper=0.489 effort=140.16 velocity=0.261799 -> lower=0.002 upper=0.489 effort=1400.16 velocity=0.261799
- joint gripper_y_right: limit lower=0.002 upper=0.489 effort=140.16 velocity=0.261799 -> lower=0.002 upper=0.489 effort=1400.16 velocity=0.261799

Commit message: non explosing version

File: rma_sb_ig/resources/robots/soto_2/soto_gripper.urdf (robot description, URDF)
Before this commit: robot soto_2_1, 25 links, 24 joints
Links:
- link left_conveyor_belt: mass 0.3 -> 2
- link right_conveyor_belt: mass 0.3 -> 2
Joints:
- joint conveyor_left_to_belt: limit lower=-2.5 upper=2.5 effort=1000 velocity=0.3 -> lower=-2.5 upper=2.5 effort=140 velocity=0.3
- joint conveyor_right_to_belt: limit lower=-2.5 upper=2.5 effort=1000 velocity=0.3 -> lower=-2.5 upper=2.5 effort=140 velocity=0.3
- joint gripper_y_left: limit lower=0.002 upper=0.489 effort=1400.16 velocity=0.261799 -> lower=0.002 upper=0.489 effort=140.16 velocity=0.261799
- joint gripper_y_right: limit lower=0.002 upper=0.489 effort=1400.16 velocity=0.261799 -> lower=0.002 upper=0.489 effort=140.16 velocity=0.261799

Commit message: no meamory leak

File: rma_sb_ig/resources/robots/soto_2/soto_gripper.urdf (robot description, URDF)
Before this commit: robot soto_2_1, 25 links, 24 joints
Links:
- removed link base_link
- link gripper_y_left_link: geometry visual mesh filename=package://soto_conveyor_gripper_1_2_description/meshes/grip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
- link gripper_y_right_link: geometry visual mesh filename=package://soto_conveyor_gripper_1_2_description/meshes/grip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
- link left_conveyor_belt: geometry collision box size=5.0 0.03 0.01; visual box size=5.0 0.03 0.01
- link manipulator_base_link: geometry visual mesh filename=package://soto_vertical_axis_2_1_description/meshes/manipul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
- link right_conveyor_belt: geometry collision box size=5.0 0.03 0.01; visual box size=5.0 0.03 0.01
Joints:
- removed joint base_footprint_to_base
- joint base_to_manipulator_base: origin xyz=0.33418 0 -0.02188 rpy=0 0 0 -> xyz=0.33418 0 0.0 rpy=0 0 0; parent base_link -> base_footprint
